File: drv-hw-interface.kicad_sch (KiCad schematic)
At the start: 2 parts, among them J4 Conn_02x03_Odd_Even

Commit message: schem: reannotate
Parts:
- renumbered R25 to R31
Changed lines of the file:
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@@
 		(on_board yes)
 		(dnp no)
-		(property "Reference" "R25"
+		(property "Reference" "R31"
 			(at 149.86 87.122 90)
 			(effects
@@
 			(project "stm32f1-battery-poc"
 				(path "/4c4b6aca-9f6a-4aac-860b-eb4aeeeecc92/78df32ab-a826-4a8a-a807-1c1832d746a2"
-					(reference "R27")
+					(reference "R33")
 					(unit 1)
 				)
 				(path "/4c4b6aca-9f6a-4aac-860b-eb4aeeeecc92/9b6644b9-5397-4892-98a5-01408259cfc5"
-					(reference "R26")
+					(reference "R32")
 					(unit 1)
 				)
 				(path "/4c4b6aca-9f6a-4aac-860b-eb4aeeeecc92/fe49d06d-7afc-4ad2-a0dc-4ccf3b57cc7d"
-					(reference "R25")
+					(reference "R31")
 					(unit 1)
 				)
@@
 		(on_board yes)
 		(dnp no)
-		(property "Reference" "#PWR055"
+		(property "Reference" "#PWR068"
 			(at 146.05 91.44 0)
 			(effects
@@
 			(project "stm32f1-battery-poc"
 				(path "/4c4b6aca-9f6a-4aac-860b-eb4aeeeecc92/78df32ab-a826-4a8a-a807-1c1832d746a2"
-					(reference "#PWR058")
+					(reference "#PWR072")
 					(unit 1)
 				)
 				(path "/4c4b6aca-9f6a-4aac-860b-eb4aeeeecc92/9b6644b9-5397-4892-98a5-01408259cfc5"
-					(reference "#PWR054")
+					(reference "#PWR070")
 					(unit 1)
 				)
 				(path "/4c4b6aca-9f6a-4aac-860b-eb4aeeeecc92/fe49d06d-7afc-4ad2-a0dc-4ccf3b57cc7d"
-					(reference "#PWR055")
+					(reference "#PWR068")
 					(unit 1)
 				)
@@
 		(dnp no)
 		(fields_autoplaced yes)
-		(property "Reference" "#PWR056"
+		(property "Reference" "#PWR069"
 			(at 154.94 101.6 0)
 			(effects
@@
 			(project "stm32f1-battery-poc"
 				(path "/4c4b6aca-9f6a-4aac-860b-eb4aeeeecc92/78df32ab-a826-4a8a-a807-1c1832d746a2"
-					(reference "#PWR059")
+					(reference "#PWR073")
 					(unit 1)
 				)
 				(path "/4c4b6aca-9f6a-4aac-860b-eb4aeeeecc92/9b6644b9-5397-4892-98a5-01408259cfc5"
-					(reference "#PWR057")
+					(reference "#PWR071")
 					(unit 1)
 				)
 				(path "/4c4b6aca-9f6a-4aac-860b-eb4aeeeecc92/fe49d06d-7afc-4ad2-a0dc-4ccf3b57cc7d"
-					(reference "#PWR056")
-					(unit 1)
-				)
+					(reference "#PWR069")
+					(unit 1)
+				)

Commit message: schem: add footprints and ordering info to BOM
Parts:
- J4: footprint (none) -> Connector_PinHeader_1.27mm:PinHeader_2x03_P1.27mm_Vertical; now left out of the parts list
- R31: footprint (none) -> Resistor_SMD:R_0402_1005Metric; Basic (none) -> Y; JLCPCB Part # (none) -> C25792; Manufacturer (none) -> Uniroyal Elec; Manufacturer Part Number (none) -> 0402WGF4702TCE
Changed lines of the file:
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@@
 		(unit 1)
 		(exclude_from_sim no)
-		(in_bom yes)
+		(in_bom no)
 		(on_board yes)
 		(dnp no)
@@
 			)
 		)
-		(property "Footprint" ""
+		(property "Footprint" "Connector_PinHeader_1.27mm:PinHeader_2x03_P1.27mm_Vertical"
 			(at 137.16 91.44 0)
 			(effects
@@
 			)
 		)
-		(property "Footprint" ""
+		(property "Footprint" "Resistor_SMD:R_0402_1005Metric"
 			(at 149.86 93.218 90)
 			(effects
@@
 			(effects
 				(font
+					(size 1.27 1.27)
+				)
+				(hide yes)
+			)
+		)
+		(property "Basic" "Y"
+			(at 149.86 91.44 90)
+			(effects
+				(font
+					(size 1.27 1.27)
+				)
+				(hide yes)
+			)
+		)
+		(property "JLCPCB Part #" "C25792"
+			(at 149.86 91.44 90)
+			(effects
+				(font
+					(size 1.27 1.27)
+				)
+				(hide yes)
+			)
+		)
+		(property "Manufacturer" "Uniroyal Elec"
+			(at 149.86 91.44 90)
+			(effects
+				(font
+					(size 1.27 1.27)
+				)
+				(hide yes)
+			)
+		)
+		(property "Manufacturer Part Number" "0402WGF4702TCE"
+			(at 149.86 91.44 90)
+			(effects
+				(font

Commit message: schem: renumber schematic
Parts:
- renumbered J4 to J10, R31 to R37
Changed lines of the file:
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@@
 		(dnp no)
 		(fields_autoplaced yes)
-		(property "Reference" "J4"
+		(property "Reference" "J10"
 			(at 138.43 85.09 0)
 			(effects
@@
 			(project "stm32f1-battery-poc"
 				(path "/4c4b6aca-9f6a-4aac-860b-eb4aeeeecc92/78df32ab-a826-4a8a-a807-1c1832d746a2"
-					(reference "J6")
+					(reference "J12")
 					(unit 1)
 				)
 				(path "/4c4b6aca-9f6a-4aac-860b-eb4aeeeecc92/9b6644b9-5397-4892-98a5-01408259cfc5"
-					(reference "J5")
+					(reference "J11")
 					(unit 1)
 				)
 				(path "/4c4b6aca-9f6a-4aac-860b-eb4aeeeecc92/fe49d06d-7afc-4ad2-a0dc-4ccf3b57cc7d"
-					(reference "J4")
+					(reference "J10")
 					(unit 1)
 				)
@@
 		(on_board yes)
 		(dnp no)
-		(property "Reference" "R31"
+		(property "Reference" "R37"
 			(at 149.86 87.122 90)
 			(effects
@@
 			(project "stm32f1-battery-poc"
 				(path "/4c4b6aca-9f6a-4aac-860b-eb4aeeeecc92/78df32ab-a826-4a8a-a807-1c1832d746a2"
-					(reference "R33")
+					(reference "R39")
 					(unit 1)
 				)
 				(path "/4c4b6aca-9f6a-4aac-860b-eb4aeeeecc92/9b6644b9-5397-4892-98a5-01408259cfc5"
-					(reference "R32")
+					(reference "R38")
 					(unit 1)
 				)
 				(path "/4c4b6aca-9f6a-4aac-860b-eb4aeeeecc92/fe49d06d-7afc-4ad2-a0dc-4ccf3b57cc7d"
-					(reference "R31")
+					(reference "R37")
 					(unit 1)
 				)
@@
 		(on_board yes)
 		(dnp no)
-		(property "Reference" "#PWR068"
+		(property "Reference" "#PWR086"
 			(at 146.05 91.44 0)
 			(effects
@@
 			(project "stm32f1-battery-poc"
 				(path "/4c4b6aca-9f6a-4aac-860b-eb4aeeeecc92/78df32ab-a826-4a8a-a807-1c1832d746a2"
-					(reference "#PWR072")
+					(reference "#PWR090")
 					(unit 1)
 				)
 				(path "/4c4b6aca-9f6a-4aac-860b-eb4aeeeecc92/9b6644b9-5397-4892-98a5-01408259cfc5"
-					(reference "#PWR070")
+					(reference "#PWR088")
 					(unit 1)
 				)
 				(path "/4c4b6aca-9f6a-4aac-860b-eb4aeeeecc92/fe49d06d-7afc-4ad2-a0dc-4ccf3b57cc7d"
-					(reference "#PWR068")
+					(reference "#PWR086")
 					(unit 1)
 				)
@@
 		(dnp no)
 		(fields_autoplaced yes)
-		(property "Reference" "#PWR069"
+		(property "Reference" "#PWR087"
 			(at 154.94 101.6 0)
 			(effects
@@
 			(project "stm32f1-battery-poc"
 				(path "/4c4b6aca-9f6a-4aac-860b-eb4aeeeecc92/78df32ab-a826-4a8a-a807-1c1832d746a2"
-					(reference "#PWR073")
+					(reference "#PWR091")
 					(unit 1)
 				)
 				(path "/4c4b6aca-9f6a-4aac-860b-eb4aeeeecc92/9b6644b9-5397-4892-98a5-01408259cfc5"
-					(reference "#PWR071")
+					(reference "#PWR089")
 					(unit 1)
 				)
 				(path "/4c4b6aca-9f6a-4aac-860b-eb4aeeeecc92/fe49d06d-7afc-4ad2-a0dc-4ccf3b57cc7d"
-					(reference "#PWR069")
-					(unit 1)
-				)
+					(reference "#PWR087")
+					(unit 1)
+				)

Commit message: schem/pcb: change jumpers to smd
Parts:
- J10: footprint Connector_PinHeader_1.27mm:PinHeader_2x03_P1.27mm_Vertical -> Connector_PinHeader_1.27mm:PinHeader_2x03_P1.27mm_Vertical_SMD
Changed lines of the file:
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@@
 			)
 		)
-		(property "Footprint" "Connector_PinHeader_1.27mm:PinHeader_2x03_P1.27mm_Vertical"
+		(property "Footprint" "Connector_PinHeader_1.27mm:PinHeader_2x03_P1.27mm_Vertical_SMD"
 			(at 137.16 91.44 0)
 			(effects
